File: pcb/mcu.kicad_sch (KiCad schematic)
At the start: 35 parts, among them Q1 MMBT2222A, SW1 SKRPABE010, SW2 SKRPABE010, U1 ESP32-S3-WROOM-1-N16R2

Commit message: Renamed and added guard ring
Parts:
- C1, C10, C2, C3, C4, C5, C7: symbol Device:C -> CRGM Passive:C_Small
- J1, TP13, TP14, TP15, TP16, TP17, TP18, TP19, TP20, TP21, TP22, TP23, TP24, TP3, TP39, TP40, TP41, TP42, TP7: value ~ -> (none)
Other:
- moved on the sheet: C1, C2, C3, C4, C5
