File: pcb/power.kicad_sch (KiCad schematic)
At the start: 32 parts, among them J2 USB_C_USB2.0_16P, U2 LM66200DRLR, U3 USBLC6-2P6, U7 AZ1084-3.3

Commit message: Renamed and added guard ring
Parts:
- removed C17: 220uF, CRGM Passive:CP_Elec_6.3x5.4, symbol CRGM Passive:C_Polarized_Small
- removed C8: 100uF, CRGM Passive:C_1206_3216Metric, symbol Device:C_Small
- added C15, C16: 47uF, CRGM Passive:C_0805_2012Metric, symbol CRGM Passive:C_Small
- C6: symbol Device:C -> CRGM Passive:C_Small
- J11: value ~ -> (none); Digikey 455-BM04B-SRSS-TBTR-ND -> 455-BM03B-SRSS-TBTR-ND; LCSC C2919601 -> C2904985; MPN BM04B-SRSS-TB -> BM03B-SRSS-TB; Mouser 306-BM04BSRSSTBTLFSN -> 306-BM03BSRSSTBTLFSN
- J12, JP1, JP2, TP10, TP12, TP25, TP26, TP27, TP28, TP4, TP60, TP8: value ~ -> (none)
Connections:
- net +3.3V: now also C15.1, C16.1
- net GND: now also C15.2, C16.2
Other:
- moved on the sheet: C11, C12, D20, D23, D24, D26, D3, J11, J12, JP1, JP2, R15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
