File: pcb/requirements.kicad_sch (KiCad schematic)
At the start: 10 parts

Commit message: Renamed and added guard ring
Parts:
- H1, H2, H3, H4, LOGO1, LOGO3: value ~ -> (none)
- LOGO2: value ~ -> (none); footprint CRGM Logos:Aquarius Logo 5mm -> CRGM Logos:Aquarius Logo 8mm
- LOGO4: value ~ -> (none); footprint CRGM Logos:Aquarius Logo 5mm -> CRGM Logos:Aquarius Logo 3.5mm
- LOGO5: value ~ -> (none); footprint CRGM Logos:Roxy 6.5mm -> CRGM Logos:Roxy 5mm
- LOGO6: value ~ -> (none); footprint CRGM Logos:Roxy 6.5mm -> CRGM Logos:Roxy 8mm
